File: 8 channel relay/modulo_relay_8canales.sch (EAGLE design)
At the start: 85 parts, among them K1 G5L, K2 G5L, K3 G5L, K4 G5L, K5 G5L, K6 G5L, K7 G5L, K8 G5L, SW1 C&K_COMPONENTS_OS102011MS2QN1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

Commit message: add schematic complete
Parts:
- SW1: value C&K_COMPONENTS_OS102011MS2QN1C&K_COMPONENTS_OS102011MS2QN1_0_0 -> Slide
Other:
- note added: "2Bit Electronic"
- note added: "@johansegura92"
- note added: "Diseñado: Johan Segura"
- note added: "Relé 8 canales con optoacopladores"
- note added: "ULN2803"
- moved on the sheet: C1, C3, C4, C5, C6, D1, D11, D12, D2, D3, D4, D5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
